File: client/hardware/hardware.kicad_sch (KiCad schematic)
At the start: 58 parts, among them J1 Screw_Terminal_01x04, J2 EXT_COM, K1 G6H-2, M1 HC-12, Q1 2N7002, SW1 ADDRESS, SW2 CHANNEL, U1 XL1509-3.3, U2 TLV1117-33, U3 ESP32-C3_SUPERMINI_SMD

Commit message: hw
Parts:
- removed R12, R23, R24: 16kΩ, JLCPCB-Kicad-Footprints:R_0805, symbol JLCPCB-Resistors:1206,10kΩ
- added R14, R4: 1kΩ, JLCPCB-Kicad-Footprints:R_0805, symbol JLCPCB-Resistors:1206,10kΩ
- renumbered R9 to R10, R10 to R11, R11 to R12, R14 to R15, R15 to R16, R16 to R17, R17 to R18, R18 to R19, R19 to R20, R20 to R21, R21 to R22, R22 to R23, R25 to R24, R26 to R25, R27 to R26, R29 to R27, R30 to R29, R31 to R30, R4 to R5, R5 to R6, R6 to R7, R7 to R8, R8 to R9
Connections:
- net +3.3V: now also SW1.5, SW1.6, SW1.7, SW1.8, SW2.10, SW2.6, SW2.7, SW2.8, SW2.9; no longer SW1.1, SW1.2, SW1.3, SW1.4, SW2.1, SW2.2, SW2.3, SW2.4, SW2.5
- net ADDR_SET: now also R4.2
- net CHANNEL_SET: now also R14.2
- net at R15.1: now also SW2.4; no longer SW2.10
- net at R23.1: now also SW2.1; no longer SW2.7
- net at R21.1, R22.1: now also SW2.2; no longer SW2.8
- net at R17.1: now also SW2.3; no longer SW2.9
- net at R11.1, R12.1: now also SW1.1; no longer SW1.6
- net at R7.1: now also SW1.2; no longer SW1.7
- net at R5.1: now also SW1.3; no longer SW1.8
- new net: R14.1, SW2.5
- new net: R4.1, SW1.4
Other:
- moved on the sheet: C7, R10, R11, R12, R15, R16, R17, R18, R19, R20, R21, R22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

Commit message: update to kicad v9
Changed lines of the file:
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@@
 (kicad_sch
-	(version 20231120)
+	(version 20250114)
 	(generator "eeschema")
-	(generator_version "8.0")
+	(generator_version "9.0")
 	(paper "A4")
 	(title_block
@@
 		)
 		(instances
-			(project ""
+			(project "hardware"
 				(path "/1baff9aa-b5e6-4f52-b652-a2b8c94bd1d3"
 					(reference "C7")
@@
 		)
 		(instances
-			(project ""
+			(project "hardware"
 				(path "/1baff9aa-b5e6-4f52-b652-a2b8c94bd1d3"
 					(reference "#PWR04")
@@
 		)
 		(instances
-			(project ""
+			(project "hardware"
 				(path "/1baff9aa-b5e6-4f52-b652-a2b8c94bd1d3"
 					(reference "R1")
@@
 		)
 		(instances
-			(project ""
+			(project "hardware"
 				(path "/1baff9aa-b5e6-4f52-b652-a2b8c94bd1d3"
 					(reference "J1")
@@
 		)
 		(instances
-			(project ""
+			(project "hardware"
 				(path "/1baff9aa-b5e6-4f52-b652-a2b8c94bd1d3"
 					(reference "TP1")
@@
 		)
 		(instances
-			(project ""
+			(project "hardware"
 				(path "/1baff9aa-b5e6-4f52-b652-a2b8c94bd1d3"
 					(reference "#PWR015")
@@
 		)
 		(instances
-			(project ""
+			(project "hardware"
 				(path "/1baff9aa-b5e6-4f52-b652-a2b8c94bd1d3"
 					(reference "TP2")
@@
 		)
 		(instances
-			(project ""
+			(project "hardware"
 				(path "/1baff9aa-b5e6-4f52-b652-a2b8c94bd1d3"
 					(reference "TP4")
@@
 		)
 		(instances
-			(project ""
+			(project "hardware"
 				(path "/1baff9aa-b5e6-4f52-b652-a2b8c94bd1d3"
 					(reference "U2")
@@
 		)
 		(instances
-			(project ""
+			(project "hardware"
 				(path "/1baff9aa-b5e6-4f52-b652-a2b8c94bd1d3"
 					(reference "TP5")
@@
 		)
 		(instances
-			(project ""
+			(project "hardware"
 				(path "/1baff9aa-b5e6-4f52-b652-a2b8c94bd1d3"
 					(reference "#PWR010")
@@
 		)
 		(instances
-			(project ""
+			(project "hardware"
 				(path "/1baff9aa-b5e6-4f52-b652-a2b8c94bd1d3"
 					(reference "#PWR08")
@@
 		)
 		(instances
-			(project ""
+			(project "hardware"
 				(path "/1baff9aa-b5e6-4f52-b652-a2b8c94bd1d3"
 					(reference "#PWR021")
@@
 		)
 		(instances
-			(project ""
+			(project "hardware"
 				(path "/1baff9aa-b5e6-4f52-b652-a2b8c94bd1d3"
 					(reference "#PWR02")
@@
 		)
 		(instances
-			(project ""
+			(project "hardware"
 				(path "/1baff9aa-b5e6-4f52-b652-a2b8c94bd1d3"
 					(reference "C6")
@@
 		)
 		(instances
-			(project ""
+			(project "hardware"
 				(path "/1baff9aa-b5e6-4f52-b652-a2b8c94bd1d3"
 					(reference "#PWR03")
@@
 		)
 		(instances
-			(project ""
+			(project "hardware"
 				(path "/1baff9aa-b5e6-4f52-b652-a2b8c94bd1d3"
 					(reference "U3")
@@
 		)
 		(instances
-			(project ""
+			(project "hardware"
 				(path "/1baff9aa-b5e6-4f52-b652-a2b8c94bd1d3"
 					(reference "#PWR019")
@@
 		)
 		(instances
-			(project ""
+			(project "hardware"
 				(path "/1baff9aa-b5e6-4f52-b652-a2b8c94bd1d3"
 					(reference "Q1")
@@
 		)
 		(instances
-			(project ""
+			(project "hardware"
 				(path "/1baff9aa-b5e6-4f52-b652-a2b8c94bd1d3"
 					(reference "K1")
@@
 		)
 		(instances
-			(project ""
+			(project "hardware"
 				(path "/1baff9aa-b5e6-4f52-b652-a2b8c94bd1d3"
 					(reference "M1")
@@
 		)
 	)
+	(embedded_fonts no)
 )

Commit message: final v1.0 hardware
Parts:
- added C8: 100nF, JLCPCB-Kicad-Footprints:C_1206, symbol JLCPCB-Capacitors:1206,100nF
- C7: value 10uF -> 100nF
- R2: value 100Ω -> 4.7kΩ
- R3: value 100kΩ -> 10kΩ
Connections:
- net BAT_MEASURE: now also C7.2
- net GND: now also R28.1, C8.2
- net at R1.1, U1.3 (FB): now also C8.1
Other:
- note added: "Gate: 1-3V"
- note added: "or 10k"
- moved on the sheet: C3, C7, D3, L1, R1, R26, R27, R28, TP1, TP3, TP6
