File: controller/hardware/hardware.kicad_pcb (KiCad board)
At the start: 2 copper layers, 57 x 52.5 mm, 28 parts, among them J1 Screw_Terminal_01x02, J2 Screw_Terminal_01x02, J3 Screw_Terminal_01x02, M1 HC-12, U1 TLV1117-33, U2 ESP32-C6-SuperMini, U3 MAX3485

Commit message: final v1.0 hardware
Parts:
- C5: value 10uF -> 100nF
- moved C5 14.8 mm to (155.0, 54.7), turned to 90 degrees
Connections:
- C5 pad 2: Net-(C5-Pad2) -> BAT_MEASURE
- R7 pad 1: Net-(C5-Pad2) -> GND
Routing:
- net Net-(C5-Pad2): track 7.49 -> 0.00 mm
- net TX1: track 17.7 -> 19.2 mm
- net RX1: track 11.9 -> 13.4 mm
- net +3.3V: vias 4 -> 13
- added copper zone on B.Cu, net +3.3V
- added copper zone on F.Cu, net +3.3V
Other:
- outline, holes or cut-outs redrawn
- board text added: "v1.0"
