File: controller/hardware/hardware.kicad_sch (KiCad schematic)
At the start: 7 parts, among them M1 HC-12, U1 TLV1117-33

Commit message: hw updates
Parts:
- added C3: 100nF, JLCPCB-Kicad-Footprints:C_1206, symbol JLCPCB-Capacitors:1206,100nF
- added C5: 10uF, JLCPCB-Kicad-Footprints:C_1206, symbol JLCPCB-Capacitors:1206,100nF
- added D1, D2, D3: SMBJ12CA, JLCPCB-Kicad-Footprints:D_SMB, symbol JLCPCB-Diodes:TVS-Bi,SMBJ13CA
- added F1, F2: BSMD1812-100-30V, MyCustom:BSMD1812-100-30V, symbol MyCustom:BSMD1812-100-30V
- added J1, J2, J3: Screw_Terminal_01x02, TerminalBlock:TerminalBlock_MaiXu_MX126-5.0-02P_1x02_P5.00mm, symbol Connector:Screw_Terminal_01x02
- added L1, L2: 10uH, JLCPCB-Kicad-Footprints:L_1206, symbol JLCPCB-Inductors:10uH,25mA
- added R1, R2, R3: 10kΩ, JLCPCB-Kicad-Footprints:R_0805, symbol JLCPCB-Resistors:1206,10kΩ
- added R5: 1MΩ, JLCPCB-Kicad-Footprints:R_0805, symbol JLCPCB-Resistors:1206,10kΩ
- added R6: 1kΩ, JLCPCB-Kicad-Footprints:R_0805, symbol JLCPCB-Resistors:1206,10kΩ
- added R7: 100kΩ, JLCPCB-Kicad-Footprints:R_0805, symbol JLCPCB-Resistors:1206,10kΩ
- added TP2: BAT_V, TestPoint:TestPoint_Pad_D1.5mm, symbol Connector:TestPoint_Probe
- added U2: ESP32-C6-SuperMini, TrailCurrentFootprints:ESP32-C6-SuperMini_SMD, symbol TrailCurrentSymbolLibrary:ESP32-C6-SuperMini
- added U3: MAX3485, Package_SO:SOIC-8_3.9x4.9mm_P1.27mm, symbol Interface_UART:MAX3485
- renumbered C3 to C4, R1 to R4
Connections:
- net +3.3V: now also C3.1, R1.1, U2.13 (3V3), U3.8 (VCC)
- net +5V: now also J1.1 (Pin_1)
- net GND: now also C3.2, C5.1, D2.1, D3.1, J1.2 (Pin_2), J2.2 (Pin_2), R2.2, R3.2, U2.12 (GND), U3.5 (GND)
- net RX: now also U2.6 (GPIO3)
- net SET: now also U2.5 (GPIO2)
- net TX: now also U2.7 (GPIO4)
- new net: C5.2, R7.1
- new net: R5.1, R6.2, R7.2
- new net: D1.1, D3.2, F1.1, R2.1, U3.6 (A)
- new net: D1.2, D2.2, F2.1, R1.2, U3.7 (B)
- new net: F1.2, L1.1
- new net: F2.2, L2.1
- new net +BATT: J2.1 (Pin_1), R5.2
- new net BAT_MEASURE: R6.1, TP2.1, U2.4 (GPIO1)
- new net RS485-1_A: J3.1 (Pin_1), L1.2
- new net RS485-1_B: J3.2 (Pin_2), L2.2
- new net RX1: U2.8 (GPIO5), U3.1 (RO)
- new net TX1: U2.9 (GPIO6), U3.4 (DI)
- new net TX1_EN: R3.1, U2.10 (GPIO7), U3.2 (~{RE}), U3.3 (DE)
Other:
- title: (none) -> Claycast controller
- moved on the sheet: C1, C2, C4, M1, R4, TP1, U1

Commit message: final v1.0 hardware
Parts:
- C5: value 10uF -> 100nF
Connections:
- net BAT_MEASURE: now also C5.2
- net GND: now also R7.1
Other:
- moved on the sheet: C5, R5, R6, R7, TP2
