File: remote/hardware/hardware.kicad_pcb (KiCad board)
At the start: 2 copper layers, 42 x 112.5 mm, 0 parts

Commit message: final v1.0 hardware
Parts:
- added C1: 10uF, PCM_JLCPCB:C_1206, B.Cu at (121.8, 78.2)
- added C2: 330uF, Capacitor_THT:CP_Radial_D6.3mm_P2.50mm, B.Cu at (108.0, 75.0)
- added C3: 10uF, PCM_JLCPCB:C_1206, F.Cu at (104.2, 54.0)
- added C4: 10uF, PCM_JLCPCB:C_1206, B.Cu at (136.3, 88.8)
- added D1: 1N4007W, Diode_SMD:D_SMB, B.Cu at (121.0, 82.5)
- added D2: LED, LED_SMD:LED_1206_3216Metric_Pad1.42x1.75mm_HandSolder, F.Cu at (121.0, 43.5)
- added J1: Antenna, Connector_PinHeader_1.00mm:PinHeader_1x01_P1.00mm_Vertical, F.Cu at (131.5, 56.0)
- added J2: BAT +, Connector_PinHeader_1.00mm:PinHeader_1x01_P1.00mm_Vertical, F.Cu at (126.5, 89.5)
- added J3: BAT -, Connector_PinHeader_1.00mm:PinHeader_1x01_P1.00mm_Vertical, F.Cu at (115.5, 89.5)
- added M1: HC-12, HC-12:MA05-1, B.Cu at (132.7, 84.0)
- added Q1: 2N7002, Package_TO_SOT_SMD:SOT-23, F.Cu at (135.3, 76.8)
- added R1: 10kΩ, JLCPCB-Kicad-Footprints:R_0805, F.Cu at (118.0, 71.0)
- added R10: 220Ω, JLCPCB-Kicad-Footprints:R_1206, F.Cu at (111.5, 43.4)
- added R2: 10kΩ, JLCPCB-Kicad-Footprints:R_0805, F.Cu at (123.8, 71.0)
- added R3: 10kΩ, JLCPCB-Kicad-Footprints:R_0805, F.Cu at (118.0, 73.8)
- added R4: 10kΩ, JLCPCB-Kicad-Footprints:R_0805, F.Cu at (123.8, 73.8)
- added R5: 10kΩ, JLCPCB-Kicad-Footprints:R_0805, F.Cu at (118.0, 76.5)
- added R6: 10kΩ, JLCPCB-Kicad-Footprints:R_0805, F.Cu at (123.8, 76.5)
- added R7: 10kΩ, JLCPCB-Kicad-Footprints:R_0805, F.Cu at (123.9, 79.2)
- added R8: 4.7kΩ, JLCPCB-Kicad-Footprints:R_0805, F.Cu at (135.2, 70.0)
- added R9: 10kΩ, JLCPCB-Kicad-Footprints:R_0805, F.Cu at (135.2, 72.8)
- added SW1: SW_Push, Button_Switch_SMD:SW_Push_1P1T_NO_E-Switch_TL3301NxxxxxG, F.Cu at (111.0, 64.0)
- added SW2: SW_Push, Button_Switch_SMD:SW_Push_1P1T_NO_E-Switch_TL3301NxxxxxG, F.Cu at (131.0, 64.0)
- added SW3: SW_Push, Button_Switch_SMD:SW_Push_1P1T_NO_E-Switch_TL3301NxxxxxG, F.Cu at (111.0, 84.0)
- added SW4: SW_Push, Button_Switch_SMD:SW_Push_1P1T_NO_E-Switch_TL3301NxxxxxG, F.Cu at (131.0, 84.0)
- added SW5: SW_Push, Button_Switch_SMD:SW_Push_1P1T_NO_E-Switch_TL3301NxxxxxG, F.Cu at (111.0, 104.0)
- added SW6: SW_Push, Button_Switch_SMD:SW_Push_1P1T_NO_E-Switch_TL3301NxxxxxG, F.Cu at (131.0, 104.0)
- added U1: TLV1117-33, Package_TO_SOT_SMD:TO-252-2, B.Cu at (108.5, 83.0)
- added U2: ESP32-C3_SUPERMINI_SMD, ESP32-C3_SUPERMINI_SMD:MODULE_ESP32-C3_SUPERMINI, B.Cu at (113.5, 57.1)
Routing:
- net +3.3V: track 0.00 -> 112.1 mm, vias 0 -> 66
- net B6: track 0.00 -> 73.9 mm, vias 0 -> 1
- net B5: track 0.00 -> 64.0 mm, vias 0 -> 1
- net B4: track 0.00 -> 45.1 mm, vias 0 -> 1
- net RX: track 0.00 -> 40.4 mm
- net B2: track 0.00 -> 40.2 mm, vias 0 -> 1
- net B3: track 0.00 -> 39.4 mm, vias 0 -> 1
- net SET: track 0.00 -> 38.7 mm, vias 0 -> 1
- net TX: track 0.00 -> 37.8 mm, vias 0 -> 2
- net B1: track 0.00 -> 27.2 mm, vias 0 -> 1
- net HC12-DRIVER: track 0.00 -> 19.3 mm, vias 0 -> 1
- net LED: track 0.00 -> 15.1 mm, vias 0 -> 1
- net +9V: track 0.00 -> 12.7 mm
- net Net-(D2-A): track 0.00 -> 9.52 mm
- net Net-(U1-VI): track 0.00 -> 6.51 mm
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- added copper zone on B.Cu, net +3.3V
- added copper zone on F.Cu, net +3.3V
- added copper zone on B.Cu, net GND
- added copper zone on F.Cu, net GND
Other:
- board text added: "ESP32C3"
- board text added: "v1.0"
