File: remote/hardware/hardware.kicad_sch (KiCad schematic)
At the start: 11 parts, among them M1 HC-12, Q1 2N7002, U1 ESP32-C3_SUPERMINI_SMD, U2 TLV1117-33

Commit message: final v1.0 hardware
Parts:
- removed TP1: 3V3, TestPoint:TestPoint_Pad_D1.5mm, symbol Connector:TestPoint_Probe
- added C2: 330uF, Capacitor_THT:CP_Radial_D6.3mm_P2.50mm, symbol Device:C_Polarized_Small
- added D1: 1N4007W, Diode_SMD:D_SMB, symbol JLCPCB-Diodes:General,1N4007W
- added D2: LED, LED_SMD:LED_1206_3216Metric_Pad1.42x1.75mm_HandSolder, symbol Device:LED
- added J1: Antenna, Connector_PinHeader_1.00mm:PinHeader_1x01_P1.00mm_Vertical, symbol Connector:Conn_01x01_Pin
- added J2: BAT +, Connector_PinHeader_1.00mm:PinHeader_1x01_P1.00mm_Vertical, symbol Connector:Conn_01x01_Pin
- added J3: BAT -, Connector_PinHeader_1.00mm:PinHeader_1x01_P1.00mm_Vertical, symbol Connector:Conn_01x01_Pin
- added R1, R2, R3, R4, R5, R6: 10kΩ, JLCPCB-Kicad-Footprints:R_0805, symbol JLCPCB-Resistors:1206,10kΩ
- added R10: 330Ω, JLCPCB-Kicad-Footprints:R_1206, symbol JLCPCB-Resistors:1206,330Ω
- added SW1, SW2, SW3, SW4, SW5, SW6: SW_Push, Button_Switch_SMD:SW_Push_1P1T_NO_E-Switch_TL3301NxxxxxG, symbol Switch:SW_Push
- R8: renamed from R2; value 100Ω -> 4.7kΩ
- R9: renamed from R3; value 100kΩ -> 10kΩ
- renumbered C2 to C3, R4 to R7, U2 to U1, U1 to U2
Connections:
- net +3.3V: now also U2.3.3 (3V3), C2.1, R1.1, R10.1, R2.2, R3.2, R4.2, R5.2, R6.2
- net +9V: now also D1.2, J2.1 (Pin_1); no longer U1.3 (VI)
- net GND: now also U2.G (GND), C2.2, J3.1 (Pin_1), SW1.2, SW2.2, SW3.2, SW4.2, SW5.2, SW6.2; no longer M1.2 (GND)
- net RX: now also U2.6 (GPIO6)
- net SET: now also U2.8 (GPIO8)
- net TX: now also U2.7 (GPIO7)
- net HC12-DRIVER: now reaches R8.1
- net HC12-DRIVER: now also U2.10 (GPIO10)
- net ANT: now reaches M1.ANT
- net ANT: now also J1.1 (Pin_1)
- net B1: now reaches U2.0 (GPIO0)
- net B1: now also R1.2, SW1.1
- net B2: now reaches U2.1 (GPIO1)
- net B2: now also R2.1, SW2.1
- net B3: now reaches U2.2 (GPIO2)
- net B3: now also R3.1, SW3.1
- net B4: now reaches U2.3 (GPIO3)
- net B4: now also R4.1, SW4.1
- net B5: now reaches U2.4 (GPIO4)
- net B5: now also R5.1, SW5.1
- net B6: now reaches U2.5 (GPIO5)
- net B6: now also R6.1, SW6.1
- net LED: now reaches U2.9 (GPIO9)
- net LED: now also D2.1 (K)
- net at Q1.3 (D): now also M1.2 (GND)
- new net: D1.1, U1.3 (VI)
- new net: D2.2 (A), R10.2
Other:
- note added: "or 10k"
- moved on the sheet: C1, C3, C4, M1, Q1, R7, R8, R9, U1, U2
